File: src/ecap5-bcarrier-xlite.kicad_pcb (KiCad board)
At the start: 4 copper layers, 161.3 x 55.2 mm, 55 parts, among them J1 DDR4_SODIMM_Board, J2 DDR4_SODIMM_Board, J3 Conn_01x04, J4 Conn_01x04, J5 USB_C_Receptacle_USB2.0_14P, J6 Conn_Coaxial, J7 Conn_Coaxial, J8 Conn_Coaxial, J9 1935161, Q1 BC846BR13, Q2 BC846BR13, SW1 RESET_SOM1, SW2 RESET_SOM2, SW3 USER1, SW4 USER1, U1 FT232RN, U2 AP7375-33SA-7

Commit message: Improve the schematic
Parts:
- added QR*****: https://github.com/ECAP5/ECAP5, ECAP5-BCARRIER-XLITE:QRCODE, B.Cu at (89.8, 119.4)
- added REF**: Logo, ECAP5-BCARRIER-XLITE:Logo, F.Cu at (80.3, 121.9)
- added REF**: WEEE-Logo_5.6x8mm_SilkScreen, Symbol:WEEE-Logo_5.6x8mm_SilkScreen, B.Cu at (224.0, 119.4)
- added REF**: ESD-Logo_8.9x8mm_SilkScreen, Symbol:ESD-Logo_8.9x8mm_SilkScreen, B.Cu at (215.4, 119.4)
- added REF**: OSHW-Logo_7.5x8mm_SilkScreen, Symbol:OSHW-Logo_7.5x8mm_SilkScreen, B.Cu at (100.3, 119.4)
- D1: value VS-30MQ040-M3/5AT -> SS34
- D9: value P4SMAJ15CA -> SMAJ15CA/TR13
- J9: value 1935161 -> WJ127-5.0-2P
- Q1, Q2: value BC846BR13 -> MMBT4401
- SW1, SW2, SW3, SW4: footprint ECAP5-BCARRIER-XLITE:SW_Push_1P1T_NO_CK_PTS125Sx73SMTR_1 -> Button_Switch_SMD:SW_Push_1P1T_NO_CK_PTS125Sx43PSMTR
- moved U2 0.20 mm to (213.4, 111.4)
- moved C1 0.19 mm to (212.8, 108.9)
- moved C2 0.19 mm to (212.8, 113.8)
- moved D2 0.11 mm to (194.6, 122.3)
- moved Q1 0.11 mm to (195.9, 117.6)
- moved Q2 0.11 mm to (199.5, 117.6)
- moved R10 0.11 mm to (198.7, 113.7)
- moved R8 0.11 mm to (195.0, 113.7)
- moved R9 0.11 mm to (196.8, 113.7)
- moved D8 0.11 mm to (196.1, 122.3)
- moved R11 0.11 mm to (200.6, 113.7)
Connections:
- net /UART.~{RXLED} renamed /USB to UART/~{RXLED}
- net /UART.~{TXLED} renamed /USB to UART/~{TXLED}
Routing:
- net /LED2: track 88.8 -> 90.0 mm
Other:
- board text added: "Rev 1.0"
- board text removed: "rev 1.0.0"
